File: harware/relay/relay.kicad_pcb (KiCad board)
At the start: 2 copper layers, 28 parts, among them J1 Conn_01x04_Socket, K1 SANYOU_SRD_Form_C, U1 GP2S700HCP, U2 L7805, U3 L7805, U4 GP2S700HCP, U5 GP2S700HCP, U6 L7805, U7 GP2S700HCP, U8 L7805

Commit message: commit final
Parts:
- removed the J1 at (65.8, 77.0)
- removed the J1 at (65.9, 56.0)
- removed the J1 at (65.8, 98.1)
- removed the J1 at (66.2, 34.5)
- removed the K1 at (78.1, 56.8)
- removed the K1 at (78.0, 98.9)
- removed the K1 at (78.4, 35.3)
- removed the K1 at (78.0, 77.8)
- removed U7: GP2S700HCP, OptoDevice:Sharp_GP2S700HCP
- removed U8: L7805, Converter_DCDC:Converter_DCDC_Murata_OKI-78SR_Vertical
- added C1: C_US, EESTN5:CAP_ELEC_8x11.5mm, F.Cu at (79.2, 106.0)
- added C2: C_US, EESTN5:CAP_ELEC_8x11.5mm, F.Cu at (98.8, 115.4)
- added C3: C, EESTN5:CAP_0.1, F.Cu at (100.6, 105.7)
- added C4: C, EESTN5:CAP_0.1, F.Cu at (79.8, 98.8)
- added J1: Conn_01x03_Pin, TerminalBlock:TerminalBlock_bornier-3_P5.08mm, B.Cu at (27.0, 56.2)
- added J2: Conn_01x03_Pin, TerminalBlock:TerminalBlock_bornier-3_P5.08mm, F.Cu at (27.0, 77.8)
- added J3: Conn_01x03_Pin, TerminalBlock:TerminalBlock_bornier-3_P5.08mm, B.Cu at (28.0, 99.7)
- added J4: Conn_01x03_Pin, TerminalBlock:TerminalBlock_bornier-3_P5.08mm, B.Cu at (28.0, 121.0)
- added J5: Screw_Terminal_01x02, TerminalBlock:TerminalBlock_bornier-2_P5.08mm, B.Cu at (73.9, 121.5)
- added J6: Conn_01x06_Pin, Connector_PinHeader_2.00mm:PinHeader_1x06_P2.00mm_Vertical, F.Cu at (111.0, 54.4)
- added J7: Conn_01x02_Pin, Connector_PinHeader_2.00mm:PinHeader_1x02_P2.00mm_Vertical, F.Cu at (74.5, 77.3)
- added J8: Conn_01x04_Pin, Connector_PinHeader_2.00mm:PinHeader_1x04_P2.00mm_Vertical, F.Cu at (109.6, 76.5)
- added K1: SANYOU_SRD_Form_C, Relay_THT:Relay_SPDT_SANYOU_SRD_Series_Form_C, F.Cu at (35.5, 51.0)
- added K2: SANYOU_SRD_Form_C, Relay_THT:Relay_SPDT_SANYOU_SRD_Series_Form_C, F.Cu at (35.5, 73.0)
- added K3: SANYOU_SRD_Form_C, Relay_THT:Relay_SPDT_SANYOU_SRD_Series_Form_C, F.Cu at (35.5, 94.5)
- added K4: SANYOU_SRD_Form_C, Relay_THT:Relay_SPDT_SANYOU_SRD_Series_Form_C, F.Cu at (35.5, 115.9)
- added Q1: MMBT2222A, Package_TO_SOT_SMD:SOT-23, B.Cu at (58.9, 57.0)
- added Q2: MMBT2222A, Package_TO_SOT_SMD:SOT-23, B.Cu at (58.9, 79.1)
- added Q3: MMBT2222A, Package_TO_SOT_SMD:SOT-23, B.Cu at (58.9, 100.5)
- added Q4: MMBT2222A, Package_TO_SOT_SMD:SOT-23, B.Cu at (58.9, 121.9)
- added R2: R, Resistor_SMD:R_0805_2012Metric, B.Cu at (62.7, 74.5)
- added R4: R, Resistor_SMD:R_0805_2012Metric, B.Cu at (62.7, 51.4)
- added R6: R, Resistor_SMD:R_0805_2012Metric, B.Cu at (62.7, 93.9)
- added R8: R, Resistor_SMD:R_0805_2012Metric, B.Cu at (62.7, 115.8)
- added SW1: SW_Nidec_CAS-120A1, Connector_PinHeader_2.00mm:PinHeader_1x03_P2.00mm_Vertical, F.Cu at (77.0, 113.8)
- D1, D2, D3, D4, D5, D6, D7, D8, R1, R3, R5, R7, U1, U4: moved to B.Cu
- U2, U3: value L7805 -> GP2S700HCP; footprint Converter_DCDC:Converter_DCDC_Murata_OKI-78SR_Vertical -> OptoDevice:Sharp_GP2S700HCP; moved to B.Cu
- U5: value GP2S700HCP -> L7805; footprint OptoDevice:Sharp_GP2S700HCP -> Converter_DCDC:Converter_DCDC_RECOM_R-78E-0.5_THT
- U6: value L7805 -> ~; footprint Converter_DCDC:Converter_DCDC_Murata_OKI-78SR_Vertical -> esp:ESP32S_38_PINES
- moved U6 59.8 mm to (89.4, 39.5)
- moved U5 49.1 mm to (89.3, 101.9), turned to -90 degrees
- moved U3 48.0 mm to (64.3, 109.1)
- moved D8 42.8 mm to (58.0, 115.9), turned to -90 degrees
- moved U2 38.9 mm to (64.3, 88.7)
- moved R3 35.4 mm to (71.2, 49.0), turned to 180 degrees
- moved D7 34.5 mm to (66.0, 102.4), turned to -90 degrees
- moved R7 31.0 mm to (71.4, 110.3), turned to 180 degrees
- moved D6 28.6 mm to (58.0, 95.5), turned to -90 degrees
- moved D5 23.2 mm to (66.9, 83.0), turned to 180 degrees
- moved D3 23.0 mm to (71.3, 44.0), turned to 180 degrees
- moved D1 22.9 mm to (58.0, 74.5), turned to -90 degrees
- moved R1 19.6 mm to (71.0, 68.4), turned to 180 degrees
- moved D2 18.9 mm to (70.1, 63.5), turned to 180 degrees
- moved R5 18.7 mm to (70.5, 89.1), turned to -90 degrees
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Connections:
- D1 pad 1: 5v -> VCC
- D2 pad 1: 22 -> GND
- D3 pad 1: 22 -> GND
- D4 pad 1: 5v -> VCC
- D5 pad 1: 22 -> GND
- D6 pad 1: 5v -> VCC
- D7 pad 1: 22 -> GND
- D8 pad 1: 5v -> VCC
- R1 pad 1: 3.3v -> giop05
- R3 pad 1: 3.3v -> giop16
- R5 pad 1: 3.3v -> giop19
- R5 pad 2: Net-(U5-A) -> Net-(U2-A)
- R7 pad 1: 3.3v -> giop23
- R7 pad 2: Net-(U7-A) -> Net-(U3-A)
- U1 pad 2: 5v -> VCC
- U2 pad 1: Net-(D1-A) -> Net-(R6-Pad1)
- U2 pad 2: Net-(U2-GND) -> VCC
- U2 pad 3: GND -> Net-(D5-A)
- U3 pad 1: Net-(D4-A) -> Net-(R8-Pad1)
- U3 pad 2: Net-(U3-GND) -> VCC
- U3 pad 3: GND -> Net-(D7-A)
- U4 pad 2: 5v -> VCC
- U5 pad 1: Net-(R6-Pad1) -> in vcc
- U5 pad 2: 5v -> GND
- U5 pad 3: Net-(D5-A) -> VCC
- U6 pad 1: Net-(D6-A) -> unconnected-(U6-3.3-Pad1)
- U6 pad 2: Net-(U6-GND) -> unconnected-(U6-EN-Pad2)
- U6 pad 3: GND -> unconnected-(U6-GIOP36-Pad3)
Routing:
- net VCC: track 0.00 -> 556.1 mm
- net Net-(J1-Pin_4): track 138.1 -> 0.00 mm
- net Net-(J1-Pin_3): track 96.4 -> 25.6 mm
- net Net-(J2-Pin_2): track 0.00 -> 28.9 mm
- net Net-(J4-Pin_2): track 0.00 -> 28.3 mm
- net Net-(J3-Pin_2): track 0.00 -> 28.1 mm
- net Net-(D8-A): track 0.00 -> 28.1 mm
- net Net-(D4-A): track 0.00 -> 27.6 mm
- net Net-(D6-A): track 0.00 -> 27.1 mm
- net 5v: track 27.1 -> 0.00 mm
- net giop23: track 0.00 -> 26.8 mm
- net Net-(D1-A): track 0.00 -> 26.6 mm
- net in vcc: track 0.00 -> 25.9 mm
- net Net-(J2-Pin_3): track 0.00 -> 25.5 mm
- net Net-(J1-Pin_2): track 52.4 -> 27.7 mm
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- added copper zone on B.Cu, net GND
Other:
- board text added: "GND"
- board text added: "VCC"
- board text added: "gnd"
- board text added: "vcc"
